File: power.kicad_sch (KiCad schematic)
At the start: 11 parts, among them J1 Conn_02x05_Odd_Even, U2 HT7333-1

Commit message: avoided silly names
Parts:
- C3, C4, C5: value 0.1uF -> 100nF
Changed lines of the file:
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@@
 			)
 		)
-		(property "Value" "0.1uF"
+		(property "Value" "100nF"
 			(at 136.906 72.39 0)
 			(effects
@@
 			)
 		)
-		(property "Value" "0.1uF"
+		(property "Value" "100nF"
 			(at 112.522 72.39 0)
 			(effects
@@
 			)
 		)
-		(property "Value" "0.1uF"
+		(property "Value" "100nF"
 			(at 112.522 87.63 0)
 			(effects
