File: dot_flipper.kicad_sch (KiCad schematic)
At the start: 50 parts, among them J1 VCC_i, J10 LATCH_o, J11 SLEEP_o, J12 GND_o, J2 SERIN, J3 SRCLK_i, J4 LATCH_i, J5 SLEEP_i, J6 GND_i, J7 VCC_o, J8 SEROUT, J9 SRCLK_o, U1 SN74LVC1G04DCKR, U10 SN74LVC1G04DCKR, U11 DRV8837CDSGR, U12 SN74LVC1G04DCKR, U13 DRV8837CDSGR, U14 SN74LVC1G04DCKR, U15 DRV8837CDSGR, U16 SN74LVC1G04DCKR, U17 DRV8837CDSGR, U2 DRV8837CDSGR, U3 7_flip_dots, U4 SN74HC595PWR, U5 SN74LVC1G04DCKR, U6 DRV8837CDSGR, U7 SN74LVC1G04DCKR, U8 DRV8837CDSGR, U9 CDSOT236-T05C

Commit message: Update Mar 7 AM
- Implemented bus architecture to transfer data to second column, and transport signals down to each pixel
- simplified schematic more
- routed first (most difficult) pixel
Parts:
- removed TP1: SEROUT, TestPoint:TestPoint_Pad_D1.0mm, symbol Connector:TestPoint
- added C17, C18, C19, C20, C21, C22, C23: 100n/16V, Capacitor_SMD:C_0603_1608Metric, symbol Device:C
Connections:
- net GND: now also C17.1, C18.1, C19.1, C20.1, C21.1, C22.1, C23.1
- net VCC: now also U11.7 (~{SLEEP}), U13.7 (~{SLEEP}), U15.7 (~{SLEEP}), U17.7 (~{SLEEP}), U6.7 (~{SLEEP}), U8.7 (~{SLEEP}), C17.2, C18.2, C19.2, C20.2, C21.2, C22.2, C23.2
- removed net SLEEP: J11.1 (Pin_1), J5.1 (Pin_1), U11.7 (~{SLEEP}), U13.7 (~{SLEEP}), U15.7 (~{SLEEP}), U17.7 (~{SLEEP}), U2.7 (~{SLEEP}), U4.13 (~{OE}), U6.7 (~{SLEEP}), U8.7 (~{SLEEP}), U9.3 (IO2)
- new net nOE: J11.1 (Pin_1), J5.1 (Pin_1), U4.13 (~{OE}), U9.3 (IO2)
Other:
- note added: "ESD protection"

Commit message: Update Mar 7 PM
All pixels routed
7x7 variant created
Parts:
- removed H1, H2: MountingHole_Pad, MountingHole:MountingHole_2.2mm_M2_Pad_Via, symbol Mechanical:MountingHole_Pad
- added FID3: Fiducial, Fiducial:Fiducial_0.5mm_Mask1.5mm, symbol Mechanical:Fiducial
- added J13: LATCH_o, Arans_Footprints:small_pad, symbol Connector:Conn_01x01_Pin
- added J14: SLEEP_o, Arans_Footprints:small_pad, symbol Connector:Conn_01x01_Pin
- C16: footprint Capacitor_SMD:C_0805_2012Metric -> Capacitor_SMD:C_0603_1608Metric
- J10, J11, J8, J9: footprint Connector_Wire:SolderWirePad_1x01_SMD_1x2mm -> Arans_Footprints:small_pad
- J12: value GND_o -> SRCLK_o; footprint Connector_Wire:SolderWirePad_1x01_SMD_1x2mm -> Arans_Footprints:small_pad
- J7: value VCC_o -> SERIN; footprint Connector_Wire:SolderWirePad_1x01_SMD_1x2mm -> Arans_Footprints:small_pad
Connections:
- net GND: no longer J12.1 (Pin_1)
- net LATCH: now also J13.1 (Pin_1)
- net SERIN: now also J7.1 (Pin_1)
- net SRCLK: now also J12.1 (Pin_1)
- net VCC: no longer J7.1 (Pin_1)
- net nOE: now also J14.1 (Pin_1)
Other:
- moved on the sheet: J10, J11, J8, J9
